File: Hardware/Avionics/Flight Computer/Barometer.kicad_sch (KiCad schematic)
At the start: 3 parts

Commit message: updated FC
Parts:
- removed A1: LPS22DFTR, Package_LGA:ST_HLGA-10_2x2mm_P0.5mm_LayoutBorder3x2y, symbol SRAD:LPS22DFTR
- removed C1, C2: 100nF, Capacitor_SMD:C_0805_2012Metric, symbol Device:C
- added C9: 100nF, symbol Device:C
- added U4: MS5611-01BA, Package_LGA:LGA-8_3x5mm_P1.25mm, symbol Sensor_Pressure:MS5611-01BA
Connections:
- net +3V3: now also C9.1, U4.1 (VDD), U4.2 (PS), U4.4 (CSB), U4.5 (CSB)
- net GND: now also C9.2, U4.3 (GND)
- net SCL: now also U4.8 (SCLK)
- net SDA: now also U4.7 (SDI/SDA)
Other:
- note added: "7Bit I2C address of BMI088 is 0x76 = 1110110 with CSB connected to VDD, 0x77 = 1110111 if connected to GND"
- note removed: "Accurate within .702 ft"
- note removed: "The 7-bit slave address (SAD) associated to the LPS22DF is 101110xb. The SDO/SA0 pin can be used to modify the less significant bit of the device address. If the SA0 pin is connected to the voltage supply, LSb is 1 (7-bit address 1011101b=5Dh), otherwise if the SA0 pin is connected to ground, the LSb value is 0 (7-bit address 1011100b=5Ch) currently connected to ground so address: 1011100b=5Ch"
- note removed: "This has been checked over and should be good"

Commit message: Final updates
Other:
- note added: "7Bit I2C address of MS5611 is 0x76 = 1110110 with CSB connected to VDD, 0x77 = 1110111 if connected to GND"
- note removed: "7Bit I2C address of BMI088 is 0x76 = 1110110 with CSB connected to VDD, 0x77 = 1110111 if connected to GND"
Changed lines of the file:
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@@
 	(generator_version "10.0")
 	(paper "A4")
-	(text "7Bit I2C address of BMI088 is 0x76 = 1110110 with CSB connected to VDD,\n					0x77 = 1110111 if connected to GND "
+	(text "7Bit I2C address of MS5611 is 0x76 = 1110110 with CSB connected to VDD,\n					0x77 = 1110111 if connected to GND "
 		(exclude_from_sim no)
 		(at 119.634 65.278 0)
