File: Hardware/Avionics/Flight Computer/IMU.kicad_sch (KiCad schematic)
At the start: 4 parts, among them U1 BNO055

Commit message: updated FC
Parts:
- removed C3: 1uF, Capacitor_SMD:C_0805_2012Metric, symbol Device:C
- removed C4, C5: 100nF, Capacitor_SMD:C_0805_2012Metric, symbol Device:C
- removed U1: BNO055, Package_LGA:LGA-28_5.2x3.8mm_P0.5mm, symbol SRAD:BNO055
- added C10, C11: 100nF, Capacitor_SMD:C_0805_2012Metric, symbol Device:C
- added U3: BMI088, Package_LGA:Bosch_LGA-16_4.5x3mm_P0.5mm_LayoutBorder7x1y_ClockwisePinNumbering, symbol Sensor_Motion:BMI088
Connections:
- net +3V3: now also C10.1, C11.1, U3.11 (VDDIO), U3.14 (~{CSB1}), U3.3 (VDD), U3.7 (PS)
- net GND: now also C10.2, C11.2, U3.10 (SDO2), U3.15 (SDO1), U3.2 (GNDA), U3.4 (GNDA), U3.6 (GNDIO)
- net SCL: now also U3.8 (SCK/SCL)
- net SDA: now also U3.9 (SDI/SDA)
- no-connect marks 6 -> 4
Other:
- note added: "Default I2C address (SDO1 LOW): 0011000b (0x18) Alternate I2C address (SDO1 HIGH): 0011001b (0x19) SDO1 is used to switch adresss of Accelerometer Gyro: Default I2C address (SDO2 LOW): 1101000b (0x68) Alternate I2C address (SDO2 HIGH): 1101001b (0x69) SDO2 is used to switch adresss of Gyroscope"
- note removed: "Default I2C address (COM3 HIGH): 0100101b (0x29) Alternate I2C address (COM3 LOW): 0101000b (0x28) COM3 is used to switch adress"

Commit message: Final updates
Parts:
- C10, C11: KiLib_Generator (none) -> SMD_2terminal_chip_molded
- U3: KiLib_Generator (none) -> package/no_lead
Changed lines of the file:
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@@
+			)
+		)
+		(property "KiLib_Generator" "SMD_2terminal_chip_molded"
+			(at 161.29 80.01 0)
+			(hide yes)
+			(show_name no)
+			(do_not_autoplace no)
+			(effects
+				(font
+					(size 1.27 1.27)
+				)
 			)
 		)
@@
 			)
 		)
+		(property "KiLib_Generator" "SMD_2terminal_chip_molded"
+			(at 152.4 80.01 0)
+			(hide yes)
+			(show_name no)
+			(do_not_autoplace no)
+			(effects
+				(font
+					(size 1.27 1.27)
+				)
+			)
+		)
 		(pin "1"
 		)
@@
 		(in_pos_files yes)
 		(dnp no)
-		(fields_autoplaced yes)
 		(property "Reference" "U3"
-			(at 141.8433 77.47 0)
+			(at 133.858 67.056 0)
 			(show_name no)
 			(do_not_autoplace no)
@@
 		)
 		(property "Value" "BMI088"
-			(at 141.8433 80.01 0)
+			(at 133.858 69.596 0)
 			(show_name no)
 			(do_not_autoplace no)
@@
 			(at 137.16 95.25 0)
 			(hide yes)
+			(show_name no)
+			(do_not_autoplace no)
+			(effects
+				(font
+					(size 1.27 1.27)
+				)
+			)
+		)
+		(property "KiLib_Generator" "package/no_lead"
+			(at 137.16 95.25 0)
+			(hide yes)
