File: Hardware/Avionics/Flight Computer/Jack_Yeulenski_Flight_Computer.kicad_pcb (KiCad board)
At the start: 2 copper layers, 53.5 x 65.5 mm, 27 parts, among them J1 SW, J2 BAT, J3 UART Radio Connector, J4 I2C GPS Connector, U1 BNO055

Commit message: PCB updates
Parts:
- added C6: 10uF, Capacitor_SMD:C_0805_2012Metric, F.Cu at (118.5, 64.0)
- added C7: 22uF, Capacitor_SMD:C_0805_2012Metric, F.Cu at (119.0, 67.5)
- added C8: 22uF, Capacitor_SMD:C_0805_2012Metric, F.Cu at (111.5, 68.0)
- added C9: 22uF, Capacitor_SMD:C_0805_2012Metric, F.Cu at (106.0, 78.0)
- added J5: SERVO_2, Connector_PinHeader_2.54mm:PinHeader_1x03_P2.54mm_Vertical, F.Cu at (106.0, 69.5)
- added L1: 1 uH, Inductor_SMD:L_Coilcraft_XAL7030-102, F.Cu at (115.5, 74.0)
- added R6: 732kOhms, Resistor_SMD:R_0603_1608Metric, F.Cu at (114.2, 59.5)
- added R7: 100kOhms, Resistor_SMD:R_0603_1608Metric, F.Cu at (113.5, 62.3)
- added U2: TPS61022, Package_DFN_QFN:Texas_RWU0007A_VQFN-7_2x2mm_P0.5mm, F.Cu at (116.0, 67.2)
- J3: value UART Radio Connector -> SERVO_1; footprint Connector_JST:JST_XH_S4B-XH-A_1x04_P2.50mm_Horizontal -> Connector_PinHeader_2.54mm:PinHeader_1x03_P2.54mm_Vertical
- moved J3 12.0 mm to (106.0, 59.0), turned to 0 degrees
- moved H1 3.04 mm to (107.0, 48.5)
- moved H4 2.55 mm to (107.5, 97.5)
- moved J4 2.50 mm to (113.4, 82.7)
Connections:
- D3 pad 2: +3V3 -> +3.3V
- J3 pad 1: +3V3 -> SERVO1_PWM
- J3 pad 2: TX -> +5V_SERVO
- J3 pad 3: RX -> GND
- J4 pad 1: +3V3 -> +3.3V
- J4 pad 2: SDA -> SDA2
- J4 pad 3: SCL -> SCL2
- Teensy4.1 pad 2: unconnected-(Teensy4.1-PWM-Pad2) -> SERVO1_PWM
- Teensy4.1 pad 24: unconnected-(Teensy4.1-SCL2-Pad24) -> SCL2
- Teensy4.1 pad 25: unconnected-(Teensy4.1-SDA2-Pad25) -> SDA2
- Teensy4.1 pad 3: unconnected-(Teensy4.1-PWM-Pad3) -> SERVO2_PWM
- Teensy4.1 pad 3V: +3V3 -> +3.3V
Routing:
- net SCL: track 143.8 -> 59.9 mm
- net SDA: track 103.0 -> 20.4 mm
- net Net-(BZ1-+): track 8.79 -> 84.3 mm
- net GND: track 258.3 -> 309.1 mm, vias 9 -> 10
- net +3V3: track 98.9 -> 48.5 mm, vias 5 -> 4
- net +5V_SERVO: track 0.00 -> 50.3 mm, vias 0 -> 2
- net Net-(J1-Pin_1): track 20.6 -> 67.6 mm, vias 2 -> 3
- net Net-(U2-FB): track 0.00 -> 32.6 mm
- net +3.3V: track 0.00 -> 27.8 mm
- net RX: track 23.1 -> 0.00 mm
- net SERVO2_PWM: track 0.00 -> 20.1 mm
- net SERVO1_PWM: track 0.00 -> 18.1 mm, vias 0 -> 1
- net TX: track 17.0 -> 0.00 mm
- net SDA2: track 0.00 -> 13.8 mm
- net SCL2: track 0.00 -> 8.66 mm
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Other:
- board size 53.5 x 65.5 mm -> 56 x 65.5 mm
- board text removed: "Radio connector"

Commit message: updated FC
Parts:
- removed A1: LPS22DFTR, Package_LGA:ST_HLGA-10_2x2mm_P0.5mm_LayoutBorder3x2y
- removed C1, C2, C4, C5: 100nF, Capacitor_SMD:C_0805_2012Metric
- removed C3: 1uF, Capacitor_SMD:C_0805_2012Metric
- removed C9: 22uF, Capacitor_SMD:C_0805_2012Metric
- removed U1: BNO055, Package_LGA:LGA-28_5.2x3.8mm_P0.5mm
- added C10: 100nF, Capacitor_SMD:C_0805_2012Metric, F.Cu at (108.0, 103.5)
- added C11: 100nF, Capacitor_SMD:C_0805_2012Metric, F.Cu at (108.0, 107.5)
- added CR1: MBRS120T3G, footprints:SDO_MBRS120T3G_OSI, F.Cu at (153.0, 62.5)
- added R10: 300, Resistor_SMD:R_0603_1608Metric, F.Cu at (144.0, 89.5)
- added R11: 110, Resistor_SMD:R_0603_1608Metric, F.Cu at (140.5, 89.5)
- added R12: 280, Resistor_SMD:R_0603_1608Metric, F.Cu at (148.8, 73.5)
- added R8: 3.3k, Resistor_SMD:R_0603_1608Metric, F.Cu at (153.0, 73.5)
- added R9: 10k, Resistor_SMD:R_0603_1608Metric, F.Cu at (146.5, 86.0)
- added U3: BMI088, Package_LGA:Bosch_LGA-16_4.5x3mm_P0.5mm_LayoutBorder7x1y_ClockwisePinNumbering, F.Cu at (147.8, 69.5)
- added U4: MS5611-01BA, Package_LGA:LGA-8_3x5mm_P1.25mm, F.Cu at (143.6, 69.1)
- C6: value 10uF -> 0.01 uF
- C7: value 22uF -> 22 uF
- J3, J5: footprint Connector_PinHeader_2.54mm:PinHeader_1x03_P2.54mm_Vertical -> Connector_JST:JST_XH_S3B-XH-A-1_1x03_P2.50mm_Horizontal
- L1: value 1 uH -> 22 uH
- R6: value 732kOhms -> 10k
- R7: value 100kOhms -> 1k
- U2: value TPS61022 -> NCV5171EDR2G; footprint Package_DFN_QFN:Texas_RWU0007A_VQFN-7_2x2mm_P0.5mm -> footprints:SOIC-8_NB_ONS
- moved U2 38.0 mm to (154.0, 69.5)
- moved R7 33.4 mm to (145.0, 73.5), turned to 0 degrees
- moved L1 32.2 mm to (144.0, 59.0), turned to -90 degrees
- moved R6 30.4 mm to (141.0, 73.8), turned to 90 degrees
- moved C6 29.0 mm to (147.5, 65.5)
- moved C7 27.9 mm to (141.4, 84.0), turned to 180 degrees
- moved C8 6.95 mm to (118.5, 68.0), turned to -90 degrees
- moved J3 5.93 mm to (111.8, 58.0), turned to -90 degrees
- moved J5 5.87 mm to (111.8, 70.0), turned to -90 degrees
- moved H3 5.59 mm to (149.5, 93.0)
Connections:
- C6 pad 1: Net-(J1-Pin_1) -> Net-(U2-VC)
- C6 pad 2: GND -> Net-(C6-Pad2)
- C7 pad 1: +5V_SERVO -> +5V
- C8 pad 1: +5V_SERVO -> Net-(J1-Pin_1)
- L1 pad 2: Net-(U2-SW) -> Net-(U2-VSW)
- R6 pad 1: +5V_SERVO -> GND
- R6 pad 2: Net-(U2-FB) -> Net-(C6-Pad2)
- R7 pad 1: Net-(U2-FB) -> GND
- R7 pad 2: GND -> Net-(R12-Pad1)
- U2 pad 1: GND -> Net-(U2-VC)
- U2 pad 2: Net-(U2-SW) -> Net-(U2-FB)
- U2 pad 3: +5V_SERVO -> unconnected-(U2-TEST-Pad3)
- U2 pad 4: Net-(U2-FB) -> unconnected-(U2-SS-Pad4)
- U2 pad 7: Net-(J1-Pin_1) -> GND
Routing:
- net +3V3: track 48.5 -> 143.1 mm, vias 4 -> 7
- net Net-(BZ1-+): track 84.3 -> 8.79 mm
- net GND: track 309.1 -> 249.1 mm, vias 10 -> 2
- net SCL: track 59.9 -> 13.9 mm, vias 1 -> 2
- net Net-(C6-Pad2): track 0.00 -> 45.4 mm
- net +5V_SERVO: track 50.3 -> 13.8 mm, vias 2 -> 0
- net +5V: track 0.00 -> 35.4 mm, vias 0 -> 2
- net Net-(U2-VSW): track 0.00 -> 24.6 mm
- net Net-(U2-FB): track 32.6 -> 8.11 mm
- net Net-(R10-Pad2): track 0.00 -> 19.4 mm
- net Net-(J1-Pin_1): track 67.6 -> 86.7 mm, vias 3 -> 1
- net Net-(U2-SW): track 8.23 -> 0.00 mm
- net SERVO1_PWM: track 18.1 -> 10.6 mm, vias 1 -> 0
- net Net-(U2-VC): track 0.00 -> 5.61 mm
- net SERVO2_PWM: track 20.1 -> 15.4 mm
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Other:
- board size 56 x 65.5 mm -> 57 x 65.5 mm
- board text added: "Jack Yeulenski Matt Urban"
- board text removed: "Jack Yeulenski"

Commit message: Final updates
Parts:
- C7, C8: footprint Capacitor_SMD:C_0805_2012Metric -> footprints:CAP_YX_5X11_RUB
- L1: footprint Inductor_SMD:L_Coilcraft_XAL7030-102 -> footprints:IND_TAIYO_NRS8040_TAY
- moved C8 19.0 mm to (115.6, 49.2)
- moved C7 3.02 mm to (141.8, 87.0), turned to 90 degrees
- moved R9 3.01 mm to (149.4, 86.8)
- moved R11 2.92 mm to (143.2, 90.6), turned to 0 degrees
- moved R10 2.56 mm to (146.4, 88.6)
- moved U2 1.91 mm to (155.4, 68.2)
- moved R8 1.80 mm to (154.8, 73.6)
- moved R12 1.78 mm to (150.6, 73.5)
- moved CR1 1.49 mm to (152.0, 61.4)
- moved H3 1.12 mm to (150.6, 92.8)
- moved L1 0.82 mm to (143.8, 58.2)
- moved U3 0.66 mm to (148.2, 69.0)
- moved H2 0.50 mm to (144.0, 49.0)
- moved U4 0.50 mm to (143.2, 68.8)
- moved J1 0.40 mm to (154.2, 56.0)
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Routing:
- net GND: track 249.1 -> 282.3 mm, vias 2 -> 4
- net Net-(J1-Pin_2): track 34.6 -> 50.4 mm, vias 2 -> 1
- net Net-(J1-Pin_1): track 86.7 -> 71.5 mm, vias 1 -> 0
- net +5V: track 35.4 -> 46.4 mm, vias 2 -> 3
- net +3V3: track 143.1 -> 133.8 mm, vias 7 -> 5
- net Net-(C6-Pad2): track 45.4 -> 51.9 mm, vias 0 -> 2
- net Net-(U2-VSW): track 24.6 -> 31.1 mm, vias 0 -> 2
- net SDA: track 24.5 -> 20.0 mm
- net +5V_SERVO: track 13.8 -> 15.9 mm, vias 0 -> 1
- net SCL: track 13.9 -> 15.9 mm, vias 2 -> 1
- net Net-(R12-Pad1): track 2.18 -> 3.95 mm
- net Net-(U2-FB): track 8.11 -> 9.56 mm
- net Net-(R10-Pad2): track 19.4 -> 18.0 mm
- net Net-(U2-VC): track 5.61 -> 4.60 mm
- net Net-(R10-Pad1): track 3.50 -> 2.86 mm
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Other:
- board size 57 x 65.5 mm -> 57.4 x 65.5 mm
